File: wedding_guestbook_hw.kicad_sch (KiCad schematic)
At the start: 4 parts, among them J1 Conn_01x04

Commit message: Updated 1x4 conn footprint assignment
Parts:
- ASSY1, ASSY2: footprint (none) -> Smart Nixie Tube:1356ST
- ASSY3: footprint (none) -> Smart Nixie Tube:1364 - HVPS
- J1: footprint (none) -> Connector_PinHeader_2.54mm:PinHeader_1x04_P2.54mm_Vertical
Changed lines of the file:
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@@
       (effects (font (size 1.27 1.27)))
     )
-    (property "Footprint" "" (at 161.29 90.17 0)
+    (property "Footprint" "Smart Nixie Tube:1364 - HVPS" (at 161.29 90.17 0)
       (effects (font (size 1.27 1.27)) hide)
     )
@@
       (effects (font (size 1.27 1.27)))
     )
-    (property "Footprint" "" (at 110.49 90.17 0)
+    (property "Footprint" "Smart Nixie Tube:1356ST" (at 110.49 90.17 0)
       (effects (font (size 1.27 1.27)) hide)
     )
@@
       (effects (font (size 1.27 1.27)))
     )
-    (property "Footprint" "" (at 135.89 90.17 0)
+    (property "Footprint" "Smart Nixie Tube:1356ST" (at 135.89 90.17 0)
       (effects (font (size 1.27 1.27)) hide)
     )
@@
       (effects (font (size 1.27 1.27)) (justify left))
     )
-    (property "Footprint" "" (at 189.23 95.25 0)
-      (effects (font (size 1.27 1.27)) hide)
-    )
+    (property "Footprint" "Connector_PinHeader_2.54mm:PinHeader_1x04_P2.54mm_Vertical" (at 189.23 95.25 0)
+      (effects (font (size 1.27 1.27)) hide)
+    )
